File: CH572D-Button/CH572D-Button.kicad_sch (KiCad schematic)
At the start: 1 part

Commit message: button done hope it works not requires enig plating for the atnenana
Parts:
- removed U1: ~, Ch572D:CH572D, symbol CH572D:CH572D
- added B1: ~, Footprint:supersmallbattery, symbol supersmallbattery:Battery
- added C1: 0.1uF, Footprint:C_0603, symbol fab:C_0603
- added C2: 1uF, Footprint:C_0603, symbol fab:C_0603
- added C5, C6: 2.2uF, Footprint:C_0603, symbol 0603:C_0603
- added C7: 0.1uF, Footprint:C_0603, symbol 0603:C_0603
- added E1: AMCA31-2R450G-S1F-T3, CHXXX:ANT-F-1-2.4G-1.6mmFR4-WCH, symbol ceramic antenna:AMCA31-2R450G-S1F-T3
- added J1: USB4105-GF-A, Footprint:usbc, symbol usbc:USB4105-GF-A
- added R1, R2: 5.1k, Footprint:R_0603, symbol fab:R_0603
- added R3: 1.5k, Footprint:R_0603, symbol 0603:R_0603
- added R4: 33k, Footprint:0603, symbol fab:R_0603
- added S1: TL3365AF180QG, Footprint:button, symbol button:TL3365AF180QG
- added U1: TCR2EF33_LMCT, Footprint:voltage regulator, symbol voltage regulator:TCR2EF33_LMCT
- added U2: ~, Footprint:CH572D, symbol CH572D:CH572D
- added U3: CPG151101D01, EasyEDA:SW-TH_CPG151101D9X, symbol EasyEDA:CPG151101D01
- added U4: TP4057_C725791, EasyEDA:SOT-23-6_L2.9-W1.6-P0.95-LS2.8-BR, symbol EasyEDA:TP4057_C725791
- added Y1: 32mhz, Footprint:32mhz crystal, symbol 32mhz crystal:XRCGB32M000F2P01R0
Connections:
- new net: B1.+, U4.3 (BAT)
- new net: R4.2, U4.6 (PROG)
- new net: E1.1, U2.5 (ANT)
- new net: R3.1, S1.3, S1.4
- new net: U2.2 (XO), Y1.3
- new net: U2.3 (XI), Y1.1
- new net: J1.A5 (CC1), R2.1
- new net: J1.B5 (CC2), R1.1
- new net Button: U2.9 (PA9/SDA/R5/TMR3), U3.1
- new net D+: J1.A6 (DP1), J1.B6 (DP2), R3.2, U2.12 (PA1/UDP/R3/T2/SDA1)
- new net D-: J1.A7 (DN1), J1.B7 (DN2), U2.11 (PA0/UDM/R2/T3/SCL1)
- new net PWR_3V3: C2.1, C6.1, C7.1, S1.1, S1.2, U1.5 (VOUT), U2.6 (VDD33), U2.7 (VIO33), U4.4 (VCC)
- new net PWR_5V: C1.2, C5.1, J1.A4_B9 (VBUS), J1.B4_A9 (VBUS__1), U1.1 (VIN), U1.3 (CONTROL), U2.8 (V5)
- new net PWR_GND: B1.-, C1.1, C2.2, C5.2, C6.2, C7.2, J1.A1_B12 (GND), J1.B1_A12 (GND__1), J1.SH1 (SHELL_GND), J1.SH2 (SHELL_GND__1), J1.SH3 (SHELL_GND__2), J1.SH4 (SHELL_GND__3), R1.2, R2.2, R4.1, U1.2 (GND), U2.21 (GND/EPAD), U3.2, U4.2 (GND)
- no-connect marks 0 -> 5
Other:
- note added: "Boot/Download button"
Changed lines of the file:
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@@
 	(generator_version "9.0")
 	(paper "A4")
-	(symbol
-		(lib_id "CH572D:CH572D")
-		(at 119.38 108.585 0)
-		(unit 1)
-		(exclude_from_sim no)
-		(in_bom yes)
-		(on_board yes)
-		(dnp no)
-		(fields_autoplaced yes)
-		(property "Reference" "U1"
-			(at 120.015 88.9 0)
-			(effects
-				(font
-					(size 1.27 1.27)
-				)
-			)
-		)
-		(property "Value" "~"
-			(at 120.015 90.17 0)
-			(effects
-				(font
-					(size 1.27 1.27)
-				)
-			)
-		)
-		(property "Footprint" "Ch572D:CH572D"
-			(at 93.98 128.143 0)
-			(effects
-				(font
-					(size 1.27 1.27)
-				)
-				(hide yes)
-			)
-		)
-		(property "Datasheet" ""
-			(at 119.38 108.585 0)
-			(effects
-				(font
-					(size 1.27 1.27)
-				)
-				(hide yes)
-			)
-		)
-		(property "Description" ""
-			(at 119.38 108.585 0)
-			(effects
-				(font
-					(size 1.27 1.27)
-				)
-				(hide yes)
-			)
-		)
-		(pin "18"
-		)
-		(pin "6"
-		)
-		(pin "8"
-		)
-		(pin "7"
-		)
-		(pin "4"
-		)
-		(pin "9"
-		)
-		(pin "3"
-		)
-		(pin "5"
-		)
-		(pin "21"
-		)
-		(pin "10"
-		)
-		(pin "16"
-		)
-		(pin "13"
-		)
-		(pin "14"
-		)
-		(pin "12"
-		)
-		(pin "1"
-		)
-		(pin "2"
-		)
-		(pin "19"
-		)
-		(pin "20"
-		)
-		(pin "17"
-		)
-		(pin "15"
-		)
-		(pin "11"
-		)
-		(instances
-			(project ""
-				(path "/3b701072-8141-40bc-9ded-8d245f000183"
-					(reference "U1")
-					(unit 1)
-				)
-			)
-		)
-	)
-	(sheet_instances
-		(path "/"
-			(page "1")
-		)
-	)
-	(embedded_fonts no)
-)
